Commit message: Basic Go2 setup (can walk in simulation)

File: legged_examples/legged_unitree/legged_unitree_description/urdf/go2/const.xacro (robot description, xacro)
@@ -12,8 +12,14 @@
     <xacro:property name="thigh_shoulder_radius" value="0.041"/>
     <xacro:property name="thigh_shoulder_length" value="0.032"/>
+    <!-- ADDED -->
+    <xacro:property name="thigh_shoulder_y_offset" value="-0.008"/>
     <xacro:property name="thigh_width" value="0.0245"/>
     <xacro:property name="thigh_height" value="0.034"/>
+    <!-- ADDED -->
+    <xacro:property name="thigh_x_offset" value="0"/>
     <xacro:property name="calf_width" value="0.016"/>
     <xacro:property name="calf_height" value="0.016"/>
+    <!-- ADDED -->
+    <xacro:property name="calf_x_offset" value="0.0"/>
     <xacro:property name="foot_radius" value="0.02"/>
     <xacro:property name="stick_radius" value="0.01"/>
